Commit message: commit on 'main'

File: environment/urdf/ur5_robotiq_140.urdf (robot description, URDF)
Before this commit: robot ur5_robotiq_140, 20 links, 19 joints
Joints:
- joint elbow_joint: limit lower=-3.14159265359 upper=3.14159265359 effort=150.0 velocity=3.15 -> lower=0 upper=3.14159265359 effort=150.0 velocity=3.15

File: environment/urdf/ur5_robotiq_85.urdf (robot description, URDF)
Before this commit: robot ur5_robotiq_85, 20 links, 19 joints
Joints:
- joint elbow_joint: limit lower=-3.14159265359 upper=3.14159265359 effort=150.0 velocity=3.15 -> lower=0 upper=3.14159265359 effort=150.0 velocity=3.15

Commit message: Reverted back to last working commit.

File: environment/urdf/ur5_robotiq_140.urdf (robot description, URDF)
Before this commit: robot ur5_robotiq_140, 20 links, 19 joints
Joints:
- joint elbow_joint: limit lower=0 upper=3.14159265359 effort=150.0 velocity=3.15 -> lower=-3.14159265359 upper=3.14159265359 effort=150.0 velocity=3.15

File: environment/urdf/ur5_robotiq_85.urdf (robot description, URDF)
Before this commit: robot ur5_robotiq_85, 20 links, 19 joints
Joints:
- joint elbow_joint: limit lower=0 upper=3.14159265359 effort=150.0 velocity=3.15 -> lower=-3.14159265359 upper=3.14159265359 effort=150.0 velocity=3.15

Commit message: commit on 'new_model'

File: environment/urdf/ur5_robotiq_140.urdf (robot description, URDF)
Before this commit: robot ur5_robotiq_140, 20 links, 19 joints
Joints:
- joint elbow_joint: limit lower=0 upper=3.14159265359 effort=150.0 velocity=3.15 -> lower=0.1 upper=3.14159265359 effort=150.0 velocity=3.15

Commit message: commit on 'new_model'

File: environment/urdf/ur5_robotiq_140.urdf (robot description, URDF)
Before this commit: robot ur5_robotiq_140, 20 links, 19 joints
Joints:
- joint shoulder_pan_joint: limit lower=-3.14159265359 upper=3.14159265359 effort=150.0 velocity=3.15 -> lower=-3.14159265359 upper=0.0 effort=150.0 velocity=3.15
